File: pcb/six_stepper_motor_driver.kicad_pcb (KiCad board)
At the start: 2 copper layers, 90 x 56 mm, 27 parts, among them J1 GPIO, M0 M0, M1 M1, M2 M2

Commit message: >:}
Connections:
- Auxillary pad 1: Net-(A6-A1) -> Net-(A6-A2)
- Auxillary pad 2: Net-(A6-A2) -> Net-(A6-A1)
- Extruder-1 pad 1: Net-(A4-A1) -> Net-(A4-A2)
- Extruder-1 pad 2: Net-(A4-A2) -> Net-(A4-A1)
- Extruder-2 pad 1: Net-(A5-A1) -> Net-(A5-A2)
- Extruder-2 pad 2: Net-(A5-A2) -> Net-(A5-A1)
- X-Motor pad 1: Net-(A1-A1) -> Net-(A1-A2)
- X-Motor pad 2: Net-(A1-A2) -> Net-(A1-A1)
- Y-Motor pad 1: Net-(A2-A1) -> Net-(A2-A2)
- Y-Motor pad 2: Net-(A2-A2) -> Net-(A2-A1)
- Z-Motor pad 1: Net-(A3-A1) -> Net-(A3-A2)
- Z-Motor pad 2: Net-(A3-A2) -> Net-(A3-A1)
Routing:
- net Net-(A3-A1): track 80.5 -> 86.4 mm, vias 9 -> 10
- net Net-(A1-A1): track 106.1 -> 109.3 mm, vias 9 -> 10
- net Net-(A5-A2): track 124.0 -> 127.0 mm, vias 1 -> 2
- net Net-(A6-A2): track 106.8 -> 109.7 mm, vias 7 -> 8
- net Net-(A6-A1): track 78.4 -> 81.1 mm
- net Net-(A5-A1): track 120.3 -> 117.8 mm
- net Net-(A1-A2): track 105.1 -> 102.6 mm
- net Net-(A2-B2): track 135.4 -> 137.8 mm
- net Net-(A2-A1): track 103.5 -> 105.7 mm
- net Net-(A4-A1): track 134.8 -> 136.3 mm
- net Net-(A4-A2): track 151.9 -> 152.8 mm
- net Net-(A3-A2): track 80.9 -> 80.2 mm
Other:
- board text added: "A2 A1 B1 B2"
- board text removed: "A2 A1 B2 B1"

Commit message: Change ports
Routing:
- net GND: track 223.7 -> 219.7 mm
- net Net-(J1-Pin_37): track 38.1 -> 39.0 mm

Commit message: Add Silkscreen and Path Changes & Optimizations
Routing:
- net Net-(A3-A1): track 86.4 -> 95.3 mm
- net Net-(A2-A1): track 105.7 -> 104.6 mm
- net Net-(A1-B2): track 95.5 -> 94.6 mm
- net Net-(A6-A2): track 109.7 -> 109.1 mm

Commit message: Change KiCad Design Files to add
Routing:
- net Net-(A3-A1): track 95.3 -> 86.4 mm
Changed lines of the file:
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@@
 		(grid_origin 100 100)
 		(pcbplotparams
-			(layerselection 0x00000000_00000000_55555555_575555f5)
+			(layerselection 0x00000000_00000000_55555555_575555ff)
 			(plot_on_all_layers_selection 0x00000000_00000000_00000000_00000000)
 			(disableapertmacros no)
@@
 			(drillshape 0)
 			(scaleselection 1)
-			(outputdirectory "")
+			(outputdirectory "gerber/")
 		)
 	)
@@
 	)
 	(segment
-		(start 147.032511 59.657489)
-		(end 146.746166 59.657489)
+		(start 148.886141 59.978173)
+		(end 147.353195 59.978173)
 		(width 0.2)
 		(layer "B.Cu")
@@
 	)
 	(segment
-		(start 151.583984 62.676016)
-		(end 148.886141 59.978173)
-		(width 0.2)
-		(layer "B.Cu")
-		(net "Net-(A3-A1)")
-	)
-	(segment
 		(start 172.75 87)
 		(end 174.75 89)
@@
 	)
 	(segment
-		(start 147.32 56.81)
-		(end 147.32 56.595686)
-		(width 0.2)
-		(layer "B.Cu")
-		(net "Net-(A3-A1)")
-	)
-	(segment
-		(start 146.065661 56.855662)
-		(end 146.505 57.295001)
-		(width 0.2)
-		(layer "B.Cu")
-		(net "Net-(A3-A1)")
-	)
-	(segment
 		(start 164.125 84.875)
 		(end 164.125 85.125)
@@
 	)
 	(segment
-		(start 146.990001 56.81)
-		(end 147.32 56.81)
-		(width 0.2)
-		(layer "B.Cu")
-		(net "Net-(A3-A1)")
-	)
-	(segment
 		(start 174.75 89)
 		(end 177.332441 89)
@@
 	)
 	(segment
-		(start 181.87 87.01)
-		(end 181.95 86.93)
+		(start 153.39 66.516452)
+		(end 151.583984 64.710436)
 		(width 0.2)
 		(layer "B.Cu")
@@
 	)
 	(segment
-		(start 145.005 57.916323)
-		(end 145.005 57.295001)
+		(start 181.87 87.01)
+		(end 181.95 86.93)
 		(width 0.2)
 		(layer "B.Cu")
@@
 	)
 	(segment
-		(start 145.444339 56.855662)
-		(end 146.065661 56.855662)
+		(start 145.852501 58.477479)
+		(end 145.084224 58.477479)
 		(width 0.2)
 		(layer "B.Cu")
@@
 	)
 	(segment
-		(start 151.583984 64.710436)
-		(end 151.583984 62.676016)
-		(width 0.2)
-		(layer "B.Cu")
-		(net "Net-(A3-A1)")
-	)
-	(segment
-		(start 147.353195 59.978173)
-		(end 147.032511 59.657489)
-		(width 0.2)
-		(layer "B.Cu")
-		(net "Net-(A3-A1)")
-	)
-	(segment
 		(start 154.15 76.25)
 		(end 153.75 75.85)
@@
 	)
 	(segment
-		(start 145.852501 58.477479)
-		(end 145.084224 58.477479)
-		(width 0.2)
-		(layer "B.Cu")
-		(net "Net-(A3-A1)")
-	)
-	(segment
 		(start 146.060661 72.5)
 		(end 146.891982 71.668678)
@@
 	)
 	(segment
-		(start 146.505 57.295001)
-		(end 146.990001 56.81)
+		(start 151.583984 62.676016)
+		(end 148.886141 59.978173)
 		(width 0.2)
 		(layer "B.Cu")
@@
 	)
 	(segment
-		(start 147.032511 59.657489)
+		(start 147.353195 59.978173)
 		(end 145.852501 58.477479)
 		(width 0.2)
@@
 	)
 	(segment
-		(start 146.746166 59.657489)
-		(end 145.005 57.916323)
-		(width 0.2)
-		(layer "B.Cu")
-		(net "Net-(A3-A1)")
-	)
-	(segment
-		(start 146.619314 55.895)
-		(end 145.180686 55.895)
-		(width 0.2)
-		(layer "B.Cu")
-		(net "Net-(A3-A1)")
-	)
-	(segment
 		(start 146.891982 71.668678)
 		(end 146.891982 69.332607)
@@
 	)
 	(segment
-		(start 145.005 57.295001)
-		(end 145.444339 56.855662)
-		(width 0.2)
-		(layer "B.Cu")
-		(net "Net-(A3-A1)")
-	)
-	(segment
-		(start 153.39 66.516452)
-		(end 151.583984 64.710436)
-		(width 0.2)
-		(layer "B.Cu")
-		(net "Net-(A3-A1)")
-	)
-	(segment
-		(start 148.886141 59.978173)
-		(end 147.353195 59.978173)
+		(start 151.583984 64.710436)
+		(end 151.583984 62.676016)
 		(width 0.2)
 		(layer "B.Cu")
@@
 		(width 0.2)
 		(layer "B.Cu")
-		(net "Net-(A3-A1)")
-	)
-	(segment
-		(start 147.32 56.595686)
-		(end 146.619314 55.895)
-		(width 0.2)
-		(layer "B.Cu")
