File: pcb/custom_3d_printer_stepper_motor_controller.kicad_pcb (KiCad board)
At the start: 2 copper layers, 90 x 80 mm, 32 parts, among them J10 1x2 Pin, J11 1x4 Pin, J2 1x4 Pin, J3 1x4 Pin, J4 1x4 Pin, J5 1x4 Pin, J6 1x2 Pin, J7 1x2 Pin, J8 1x2 Pin, J9 1x4 Pin, M1 Fan, Q1 M0, Q2 M1, Q3 M2, SW1 Switch, U1 5V Regulator

Commit message: Add Firmware
Other:
- board text added: "DRV8825"
- board text added: "E"
- board text added: "X"
- board text added: "Y"
- board text added: "Z"
Changed lines of the file:
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@@
 			(at 6.35 20.27 90)
 			(layer "F.SilkS")
+			(hide yes)
 			(effects
 				(font
@@
 			(at 6.35 20.27 270)
 			(layer "F.SilkS")
+			(hide yes)
 			(effects
 				(font
@@
 			(at 6.35 20.27 90)
 			(layer "F.SilkS")
+			(hide yes)
 			(effects
 				(font
@@
 		(layer "Edge.Cuts")
 	)
+	(gr_text "E"
+		(at 140 58.6 0)
+		(layer "F.SilkS")
+		(effects
+			(font
+				(size 1 1)
+				(thickness 0.15)
+			)
+			(justify left bottom)
+		)
+	)
+	(gr_text "E"
+		(at 140 70 0)
+		(layer "F.SilkS")
+		(effects
+			(font
+				(size 1 1)
+				(thickness 0.15)
+			)
+			(justify left bottom)
+		)
+	)
+	(gr_text "E"
+		(at 140 81.4 0)
+		(layer "F.SilkS")
+		(effects
+			(font
+				(size 1 1)
+				(thickness 0.15)
+			)
+			(justify left bottom)
+		)
+	)
+	(gr_text "Z"
+		(at 140 92.8 0)
+		(layer "F.SilkS")
+		(effects
+			(font
+				(size 1 1)
+				(thickness 0.15)
+			)
+			(justify left bottom)
+		)
+	)
+	(gr_text "E"
+		(at 140 104.4 0)
+		(layer "F.SilkS")
+		(effects
+			(font
+				(size 1 1)
+				(thickness 0.15)
+			)
+			(justify left bottom)
+		)
+	)
+	(gr_text "X"
+		(at 228.8 57.4 0)
+		(layer "F.SilkS")
+		(effects
+			(font
+				(size 1 1)
+				(thickness 0.15)
+			)
+			(justify left bottom)
+		)
+	)
+	(gr_text "X"
+		(at 228.8 68.8 0)
+		(layer "F.SilkS")
+		(effects
+			(font
+				(size 1 1)
+				(thickness 0.15)
+			)
+			(justify left bottom)
+		)
+	)
+	(gr_text "Y"
+		(at 228.8 80.2 0)
+		(layer "F.SilkS")
+		(effects
+			(font
+				(size 1 1)
+				(thickness 0.15)
+			)
+			(justify left bottom)
+		)
+	)
+	(gr_text "Y"
+		(at 228.8 91.6 0)
+		(layer "F.SilkS")
+		(effects
+			(font
+				(size 1 1)
+				(thickness 0.15)
+			)
+			(justify left bottom)
+		)
+	)
+	(gr_text "Z"
+		(at 228.8 102.8 0)
+		(layer "F.SilkS")
+		(effects
+			(font
+				(size 1 1)
+				(thickness 0.15)
+			)
+			(justify left bottom)
+		)
+	)
 	(gr_text "Q1\n"
 		(at 178.6 111.6 0)
@@
 		(layer "F.SilkS")
 		(effects
+			(font
+				(size 1 1)
+				(thickness 0.15)
+			)
+		)
+	)
+	(gr_text "DRV8825\n"
+		(at 168.4 97.6 270)
+		(layer "F.SilkS")
+		(effects
+			(font
+				(size 1 1)
+				(thickness 0.15)
+			)
+		)
+	)
+	(gr_text "DRV8825\n"
+		(at 168.6 63.8 270)
+		(layer "F.SilkS")
+		(effects
+			(font
+				(size 1 1)
+				(thickness 0.15)
+			)
+		)
+	)
+	(gr_text "DRV8825\n"
+		(at 168.6 80.8 270)
+		(layer "F.SilkS")
+		(effects
